Commit message: 1.add Collision radius； 2.Parameter adjustment, superior simulation effect

File: src/Gazebo/sentry_gazebo/urdf/xacro/property.xacro (robot description, xacro)
@@ -30,5 +30,5 @@
     <xacro:property name="PI" value="3.14159" />
     <xacro:property name="car_length" value="0.6" />
-    <xacro:property name="car_width" value="0.6" />
+    <xacro:property name="car_width" value="0.55" />
     <xacro:property name="car_height" value="0.16" />
     <!-- 轮胎尺寸 -->

File: src/Gazebo/sentry_gazebo/urdf/xacro/robot.urdf.xacro (robot description, xacro)
@@ -15,11 +15,11 @@
     </joint>
     <xacro:VLP-16 parent="vehicle" name="velodyne" topic="/velodyne_points" hz="10"
-        min_range="0.4" samples="350" collision_range="0.5" organize_cloud="true" gpu="false"
-        min_angle="0" max_angle="3.14159" vmin_angle="${-7/180*PI}" vmax_angle="${52/180*PI}">
+        min_range="0.2" samples="350" collision_range="0.2" organize_cloud="true" gpu="false"
+        min_angle="-0.3" max_angle="3.44159" vmin_angle="${-7/180*PI}" vmax_angle="${52/180*PI}">
         <origin xyz="0.0 0.2 ${car_height/2+0.02}" rpy="0 0 0" />
     </xacro:VLP-16>
     <xacro:VLP-16 parent="vehicle" name="velodyne2" topic="/velodyne_points2" hz="10"
-        min_range="0.4" samples="350" collision_range="0.5" organize_cloud="true" gpu="false"
-        min_angle="-3.14159" max_angle="0" vmin_angle="${-7/180*PI}" vmax_angle="${52/180*PI}">
+        min_range="0.2" samples="350" collision_range="0.2" organize_cloud="true" gpu="false"
+        min_angle="-3.44159" max_angle="0.3" vmin_angle="${-7/180*PI}" vmax_angle="${52/180*PI}">
         <origin xyz="0.0 -0.2 ${car_height/2+0.02}" rpy="0 0 0" />
     </xacro:VLP-16>

Commit message: xingtian

File: src/Gazebo/sentry_gazebo/urdf/xacro/property.xacro (robot description, xacro)
@@ -1,4 +1,3 @@
 <robot xmlns:xacro="http://www.ros.org/wiki/xacro" name="robot">
-    <xacro:property name="ns" value="$(arg ns)/" />
     <!-- 惯性矩阵 -->
     <!-- sphere球体 -->

File: src/Gazebo/sentry_gazebo/urdf/xacro/robot.urdf.xacro (robot description, xacro)
@@ -8,7 +8,7 @@
     <xacro:include filename="camera.urdf.xacro" />
     <!-- <xacro:include filename="laser.urdf.xacro" /> -->
-    <joint name="${ns}camera2base_link" type="fixed">
-        <parent link="${ns}vehicle" />
-        <child link="${ns}camera" />
+    <joint name="camera2base_link" type="fixed">
+        <parent link="vehicle" />
+        <child link="camera" />
         <origin xyz="0.2 0 0.12" rpy="0 0 0" />
         <axis xyz="0 0 0" />

File: src/Gazebo/velodyne_simulator/velodyne_description/urdf/VLP-16.urdf.xacro (robot description, xacro)
@@ -4,10 +4,10 @@
   <xacro:macro name="VLP-16"
     params="*origin parent:=base_link name:=velodyne topic:=/velodyne_points organize_cloud:=false hz:=10 lasers:=16 samples:=1875 collision_range:=0.5 min_range:=0.6 max_range:=30.0 noise:=0.008 min_angle:=-${M_PI} max_angle:=${M_PI} gpu:=false vmin_angle:=-${M_PI} vmax_angle:=${M_PI}">
-    <joint name="${ns}${name}_base_mount_joint" type="fixed">
+    <joint name="${name}_base_mount_joint" type="fixed">
       <xacro:insert_block name="origin" />  <!--插入参数宏，对应第一个参数*origin-->
-      <parent link="${ns}${parent}" />
-      <child link="${ns}${name}_base_link" />
+      <parent link="${parent}" />
+      <child link="${name}_base_link" />
     </joint>
-    <link name="${ns}${name}_base_link">
+    <link name="${name}_base_link">
       <inertial>
         <mass value="0.83" />
@@ -34,10 +34,10 @@
       </collision>
     </link>
-    <joint name="${ns}${name}_base_scan_joint" type="fixed">
+    <joint name="${name}_base_scan_joint" type="fixed">
       <origin xyz="0 0 0.0377" rpy="0 0 0" />
-      <parent link="${ns}${name}_base_link" />
-      <child link="${ns}${name}" />
+      <parent link="${name}_base_link" />
+      <child link="${name}" />
     </joint>
-    <link name="${ns}${name}">
+    <link name="${name}">
       <inertial>
         <mass value="0.01" />
@@ -53,5 +53,5 @@
     </link>
     <!-- Gazebo requires the velodyne_gazebo_plugins package -->
-    <gazebo reference="${ns}${name}">
+    <gazebo reference="${name}">
       <xacro:if value="${gpu}">
         <sensor type="gpu_ray" name="${name}-VLP16">
@@ -86,6 +86,6 @@
           </ray>
           <plugin name="gazebo_ros_laser_controller" filename="libgazebo_ros_velodyne_gpu_laser.so">
-            <topicName>/${ns}${topic}</topicName>
-            <frameName>/${ns}${name}</frameName>
+            <topicName>/${topic}</topicName>
+            <frameName>/${name}</frameName>
             <organize_cloud>${organize_cloud}</organize_cloud>
             <min_range>${min_range}</min_range>
@@ -127,6 +127,6 @@
           </ray>
           <plugin name="gazebo_ros_laser_controller" filename="libgazebo_ros_velodyne_laser.so">
-            <topicName>/${ns}${topic}</topicName>
-            <frameName>/${ns}${name}</frameName>
+            <topicName>/${topic}</topicName>
+            <frameName>/${name}</frameName>
             <organize_cloud>${organize_cloud}</organize_cloud>
             <min_range>${min_range}</min_range>
